File: KiCad/TrackController/TrackController.kicad_sch (KiCad schematic)
At the start: 22 parts, among them J1 DE9_Plug_MountingHoles, J3 Barrel_Jack_Switch, SW1 SW_Push, SW2 SW_Push, SW3 SW_Push, SW4 SW_Push, U1 TXS0108EPW

Commit message: Added KiCad design
Other:
- title: (none) -> TrackController
Changed lines of the file:
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@@
 	(generator_version "8.0")
 	(paper "A4")
+	(title_block
+		(title "TrackController")
+		(date "2024-04-29")
+		(rev "A")
+		(comment 1 "Complete Schematics")
+		(comment 2 "Design by Gerard Harkema")
+	)
 	(junction
 		(at 259.08 119.38)
