File: KiCad/TrackControllerRevB/TrackControllerRevB.kicad_pcb (KiCad board)
At the start: 2 copper layers, 130 x 60 mm, 24 parts, among them J1 DE9_Plug_MountingHoles, J3 Barrel_Jack_Switch, SW1 SW_Push, SW2 SW_Push, SW3 SW_Push, SW4 SW_Push, U1 TXS0108EPW

Commit message: 20240508
Connections:
- net /CAN-INT* renamed /CAN-INT*/TRACK-PROG-POWER-ENABLE
- net /TRACK-PULSE-H-PROG renamed /TRACK-PROG-PULSE
- net /TRACK-PULSE-H-PROG-TTL renamed /TRACK-PROG-PULSE-TTL
- CAN-MODULE1 pad 1: /CAN-INT-TTL* -> /CAN-INT*/TRACK-PROG-POWER-ENABLE-TTL
- MOTOR-SHIELD1 pad J1-7: /TRACK-ENABLE-TTL -> /CAN-INT*/TRACK-PROG-POWER-ENABLE-TTL
- U1 pad 15: /CAN-INT-TTL* -> /CAN-INT*/TRACK-PROG-POWER-ENABLE-TTL
Routing:
- net /VCC: track 0.00 -> 152.0 mm, vias 0 -> 2
- net /18V: track 0.00 -> 151.0 mm
- net /TEMP: track 0.00 -> 142.6 mm, vias 0 -> 1
- net /3V3: track 0.00 -> 129.9 mm
- net /IS: track 0.00 -> 124.4 mm
- net /RESET*: track 0.00 -> 100.1 mm, vias 0 -> 1
- net /SPARE-SWITCH-1: track 0.00 -> 98.8 mm, vias 0 -> 2
- net /MEASUREMENT_TOGGLE: track 0.00 -> 86.7 mm, vias 0 -> 1
- net /SPARE-SWITCH-2: track 0.00 -> 81.8 mm
- net /TRACK-PULSE-L: track 0.00 -> 75.7 mm
- net /TRACK-POWER-ENABLE: track 0.00 -> 60.0 mm, vias 0 -> 1
- net /TRACK-ENABLE-TTL: track 0.00 -> 53.5 mm
- net /VOLTAGE: track 0.00 -> 52.2 mm
- net /TRACK-PROG-PULSE: track 0.00 -> 51.8 mm
- net /TRACK-PULSE-H: track 0.00 -> 47.8 mm
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