File: KiCad/TrackControllerRevB/TrackControllerRevB.kicad_sch (KiCad schematic)
At the start: 22 parts, among them J1 DE9_Plug_MountingHoles, J3 Barrel_Jack_Switch, SW1 SW_Push, SW2 SW_Push, SW3 SW_Push, SW4 SW_Push, U1 TXS0108EPW

Commit message: 20240508
Connections:
- net TRACK-ENABLE-TTL: no longer MOTOR-SHIELD1.J1-7 (PWM-B)
- net CAN-INT* renamed CAN-INT*/TRACK-PROG-POWER-ENABLE
- net CAN-INT-TTL* renamed CAN-INT*/TRACK-PROG-POWER-ENABLE-TTL
- net CAN-INT*/TRACK-PROG-POWER-ENABLE-TTL: now also MOTOR-SHIELD1.J1-7 (PWM-B)
- net TRACK-PULSE-H-PROG renamed TRACK-PROG-PULSE
- net TRACK-PULSE-H-PROG-TTL renamed TRACK-PROG-PULSE-TTL
Other:
- moved on the sheet: CAN-MODULE1, ESP32, IBT_2, J1, R1, U1

Commit message: 2040514
Connections:
- net 3V3: no longer IBT_2.7 (VCC)
- net TRACK-ENABLE-TTL: now also IBT_2.3 (L-EN), IBT_2.4 (R-EN)
- net TRACK-POWER-ENABLE: no longer IBT_2.3 (L-EN), IBT_2.4 (R-EN)
- net TRACK-PULSE-L: no longer IBT_2.2 (R-PWM)
- net VCC: now also IBT_2.7 (VCC)
- net CAN-CS* renamed CAN-CS*/TRACK-PULSE-L
- net CAN-CS-TTL* renamed CAN-CS*/TRACK-PULSE-L-TTL
- net CAN-CS*/TRACK-PULSE-L-TTL: now also IBT_2.2 (R-PWM)
Changed lines of the file:
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@@
 		)
 	)
-	(label "TRACK-PULSE-L"
+	(label "CAN-CS*{slash}TRACK-PULSE-L-TTL"
 		(at 210.82 77.47 0)
 		(fields_autoplaced yes)
@@
 		)
 	)
-	(label "TRACK-POWER-ENABLE"
+	(label "TRACK-ENABLE-TTL"
 		(at 210.82 80.01 0)
 		(fields_autoplaced yes)
@@
 		)
 	)
-	(label "3V3"
+	(label "VCC"
 		(at 187.96 85.09 180)
 		(fields_autoplaced yes)
@@
 		)
 	)
-	(label "CAN-CS-TTL*"
+	(label "CAN-CS*{slash}TRACK-PULSE-L-TTL"
 		(at 224.79 41.91 0)
 		(fields_autoplaced yes)
@@
 		)
 	)
-	(label "TRACK-POWER-ENABLE"
+	(label "TRACK-ENABLE-TTL"
 		(at 187.96 80.01 180)
 		(fields_autoplaced yes)
@@
 		)
 	)
-	(label "CAN-CS*"
+	(label "CAN-CS*{slash}TRACK-PULSE-L"
 		(at 204.47 41.91 180)
 		(fields_autoplaced yes)
@@
 		)
 	)
-	(label "CAN-CS*"
+	(label "CAN-CS*{slash}TRACK-PULSE-L"
 		(at 115.57 34.29 180)
 		(fields_autoplaced yes)
@@
 		)
 	)
-	(label "CAN-CS-TTL*"
+	(label "CAN-CS*{slash}TRACK-PULSE-L-TTL"
 		(at 119.38 128.27 180)
 		(fields_autoplaced yes)
